File: KiCad/Nav/Nav.kicad_pcb (KiCad board)
At the start: 2 copper layers, 120.1 x 99.3 mm, 46 parts, among them J1 Wuerth_7499010121A, J2 Screw_Terminal_01x04, J3 B Micro USB, J4 Chassis, J5 +5v In Gnd, J6 Rx2 Tx2 Gnd, U1 3.3V Reg, U2 5.0V Reg, U3 Teensy 4.1, U4 Ada BNO085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

Commit message: kicad update
Parts:
- R5: footprint Resistor_THT:R_Axial_DIN0204_L3.6mm_D1.6mm_P2.54mm_Vertical -> Resistor_THT:R_Axial_DIN0207_L6.3mm_D2.5mm_P10.16mm_Horizontal
- U7: value MCP6002 -> MCP6002-xP
- moved J6 8.89 mm to (187.6, 124.2)
- moved R5 7.76 mm to (194.0, 125.0)
- moved D7 1.84 mm to (209.3, 125.0)
Routing:
- net Net-(J6-Pad1): track 4.97 -> 13.2 mm
- net Net-(U6-Pad18): track 3.74 -> 11.7 mm
- net Net-(J6-Pad2): track 6.54 -> 8.25 mm
Other:
- board size 120.1 x 99.3 mm -> 116.7 x 99.3 mm
