File: KiCad/Nav/Nav.kicad_sch (KiCad schematic)
At the start: 46 parts, among them J1 Wuerth_7499010121A, J2 Screw_Terminal_01x04, J3 B Micro USB, J4 Chassis, J5 +5v In Gnd, J6 Rx2 Tx2 Gnd, U1 3.3V Reg, U2 5.0V Reg, U3 Teensy 4.1, U4 Ada BNO085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

Commit message: kicad update
Parts:
- removed J5: +5v In Gnd, Connector_PinHeader_2.54mm:PinHeader_1x03_P2.54mm_Vertical, symbol Connector:Conn_01x03_Male
- added J?: WAS Terminal, TerminalBlock_TE-Connectivity:TerminalBlock_TE_282834-4_1x04_P2.54mm_Horizontal, symbol Connector:Screw_Terminal_01x04
- J2: footprint TerminalBlock_Phoenix:TerminalBlock_Phoenix_MKDS-1,5-4-5.08_1x04_P5.08mm_Horizontal -> TerminalBlock_TE-Connectivity:TerminalBlock_TE_282834-4_1x04_P2.54mm_Horizontal
- R5: footprint Resistor_THT:R_Axial_DIN0204_L3.6mm_D1.6mm_P2.54mm_Vertical -> Resistor_THT:R_Axial_DIN0207_L6.3mm_D2.5mm_P10.16mm_Horizontal
Connections:
- net +5V: now also J?.1 (Pin_1)
- net GND: now also J?.3 (Pin_3), J?.4 (Pin_4)
- net at RV1.1, RV1.2: now also J?.2 (Pin_2)
Changed lines of the file:
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@@
   (junction (at 241.3 146.05) (diameter 0) (color 0 0 0 0)
+  )
+  (junction (at 278.13 27.94) (diameter 0) (color 0 0 0 0)
   )
   (junction (at 81.28 167.64) (diameter 0) (color 0 0 0 0)
@@
     (stroke (width 0) (type default) (color 0 0 0 0))
   )
+  (wire (pts (xy 278.13 26.67) (xy 278.13 27.94))
+    (stroke (width 0) (type default) (color 0 0 0 0))
+  )
   (wire (pts (xy 217.17 22.86) (xy 220.98 22.86))
     (stroke (width 0) (type default) (color 0 0 0 0))
@@
     (stroke (width 0) (type default) (color 0 0 0 0))
   )
-  (wire (pts (xy 275.59 26.67) (xy 281.94 26.67))
-    (stroke (width 0) (type default) (color 0 0 0 0))
-  )
   (wire (pts (xy 124.46 128.27) (xy 125.73 128.27))
     (stroke (width 0) (type default) (color 0 0 0 0))
@@
     (stroke (width 0) (type default) (color 0 0 0 0))
   )
-  (wire (pts (xy 281.94 26.67) (xy 281.94 27.94))
-    (stroke (width 0) (type default) (color 0 0 0 0))
-  )
   (wire (pts (xy 215.9 118.11) (xy 226.06 118.11))
     (stroke (width 0) (type default) (color 0 0 0 0))
@@
     (stroke (width 0) (type default) (color 0 0 0 0))
   )
+  (wire (pts (xy 275.59 27.94) (xy 278.13 27.94))
+    (stroke (width 0) (type default) (color 0 0 0 0))
+  )
   (wire (pts (xy 147.32 106.68) (xy 147.32 109.22))
     (stroke (width 0) (type default) (color 0 0 0 0))
@@
     (stroke (width 0) (type default) (color 0 0 0 0))
   )
+  (wire (pts (xy 278.13 27.94) (xy 281.94 27.94))
+    (stroke (width 0) (type default) (color 0 0 0 0))
+  )
   (wire (pts (xy 243.84 146.05) (xy 250.19 146.05))
     (stroke (width 0) (type default) (color 0 0 0 0))
@@
   )
   (wire (pts (xy 128.27 130.81) (xy 128.27 132.08))
+    (stroke (width 0) (type default) (color 0 0 0 0))
+  )
+  (wire (pts (xy 275.59 26.67) (xy 275.59 27.94))
     (stroke (width 0) (type default) (color 0 0 0 0))
   )
@@
     (pin "1")
   )
-  (symbol (lib_id "Connector:Conn_01x03_Male") (at 273.05 21.59 270) (unit 1)
-    (in_bom yes) (on_board yes)
-    (property "Reference" "J5" (id 0) (at 267.97 26.67 0)
-      (effects (font (size 1.27 1.27)) (justify right))
-    )
-    (property "Value" "+5v In Gnd" (id 1) (at 278.6187 20.2574 90)
-      (effects (font (size 1.27 1.27)) (justify right))
-    )
-    (property "Footprint" "Connector_PinHeader_2.54mm:PinHeader_1x03_P2.54mm_Vertical" (id 2) (at 273.05 21.59 0)
+  (symbol (lib_id "Device:C_Small") (at 252.73 149.86 0) (unit 1)
+    (in_bom yes) (on_board yes)
+    (property "Reference" "C3" (id 0) (at 252.8264 148.1667 0)
+      (effects (font (size 1.27 1.27)) (justify left))
+    )
+    (property "Value" "0.1uF" (id 1) (at 253.0033 151.9392 0)
+      (effects (font (size 1.27 1.27)) (justify left))
+    )
+    (property "Footprint" "Capacitor_THT:C_Disc_D7.0mm_W2.5mm_P5.00mm" (id 2) (at 252.73 149.86 0)
+      (effects (font (size 1.27 1.27)) hide)
+    )
+    (property "Datasheet" "~" (id 3) (at 252.73 149.86 0)
+      (effects (font (size 1.27 1.27)) hide)
+    )
+    (pin "1")
+    (pin "2")
+  )
+  (symbol (lib_id "Connector:Screw_Terminal_01x04") (at 273.05 21.59 90) (unit 1)
+    (in_bom yes) (on_board yes) (fields_autoplaced)
+    (property "Reference" "J?" (id 0) (at 274.32 15.24 90))
+    (property "Value" "WAS Terminal" (id 1) (at 274.32 17.78 90))
+    (property "Footprint" "TerminalBlock_TE-Connectivity:TerminalBlock_TE_282834-4_1x04_P2.54mm_Horizontal" (id 2) (at 273.05 21.59 0)
       (effects (font (size 1.27 1.27)) hide)
     )
@@
     (pin "2")
     (pin "3")
-  )
-  (symbol (lib_id "Device:C_Small") (at 252.73 149.86 0) (unit 1)
-    (in_bom yes) (on_board yes)
-    (property "Reference" "C3" (id 0) (at 252.8264 148.1667 0)
-      (effects (font (size 1.27 1.27)) (justify left))
-    )
-    (property "Value" "0.1uF" (id 1) (at 253.0033 151.9392 0)
-      (effects (font (size 1.27 1.27)) (justify left))
-    )
-    (property "Footprint" "Capacitor_THT:C_Disc_D7.0mm_W2.5mm_P5.00mm" (id 2) (at 252.73 149.86 0)
-      (effects (font (size 1.27 1.27)) hide)
-    )
-    (property "Datasheet" "~" (id 3) (at 252.73 149.86 0)
-      (effects (font (size 1.27 1.27)) hide)
-    )
-    (pin "1")
-    (pin "2")
+    (pin "4")
   )
   (symbol (lib_id "power:GND") (at 217.17 57.15 0) (unit 1)
@@
     (pin "1")
   )
+  (symbol (lib_id "Device:R") (at 81.28 147.32 90) (unit 1)
+    (in_bom yes) (on_board yes)
+    (property "Reference" "R5" (id 0) (at 81.28 144.78 90))
+    (property "Value" "1k" (id 1) (at 81.28 149.86 90))
+    (property "Footprint" "Resistor_THT:R_Axial_DIN0207_L6.3mm_D2.5mm_P10.16mm_Horizontal" (id 2) (at 81.28 149.098 90)
+      (effects (font (size 1.27 1.27)) hide)
+    )
+    (property "Datasheet" "~" (id 3) (at 81.28 147.32 0)
+      (effects (font (size 1.27 1.27)) hide)
+    )
+    (pin "1")
+    (pin "2")
+  )
   (symbol (lib_id "power:GND") (at 90.17 62.23 0) (unit 1)
     (in_bom yes) (on_board yes)
@@
     (property "Reference" "J2" (id 0) (at 190.5 115.57 0))
     (property "Value" "Screw_Terminal_01x04" (id 1) (at 190.5 118.11 0))
-    (property "Footprint" "TerminalBlock_Phoenix:TerminalBlock_Phoenix_MKDS-1,5-4-5.08_1x04_P5.08mm_Horizontal" (id 2) (at 190.5 127 0)
+    (property "Footprint" "TerminalBlock_TE-Connectivity:TerminalBlock_TE_282834-4_1x04_P2.54mm_Horizontal" (id 2) (at 190.5 127 0)
       (effects (font (size 1.27 1.27)) hide)
     )
@@
     (pin "1")
   )
-  (symbol (lib_id "Device:R") (at 81.28 147.32 90) (unit 1)
-    (in_bom yes) (on_board yes)
-    (property "Reference" "R5" (id 0) (at 81.28 144.78 90))
-    (property "Value" "1k" (id 1) (at 81.28 149.86 90))
-    (property "Footprint" "Resistor_THT:R_Axial_DIN0204_L3.6mm_D1.6mm_P2.54mm_Vertical" (id 2) (at 81.28 149.098 90)
-      (effects (font (size 1.27 1.27)) hide)
-    )
-    (property "Datasheet" "~" (id 3) (at 81.28 147.32 0)
-      (effects (font (size 1.27 1.27)) hide)
-    )
-    (pin "1")
-    (pin "2")
-  )
   (symbol (lib_id "Device:C_Small") (at 152.4 104.14 0) (unit 1)
     (in_bom yes) (on_board yes)
@@
     )
     (path "/6f799b2c-1c44-4ce5-afc7-772ba3234006"
-      (reference "J2") (unit 1) (value "Screw_Terminal_01x04") (footprint "TerminalBlock_Phoenix:TerminalBlock_Phoenix_MKDS-1,5-4-5.08_1x04_P5.08mm_Horizontal")
+      (reference "J2") (unit 1) (value "Screw_Terminal_01x04") (footprint "TerminalBlock_TE-Connectivity:TerminalBlock_TE_282834-4_1x04_P2.54mm_Horizontal")
     )
     (path "/b0535057-09f3-4d30-9148-d7c69aa283c7"
@@
       (reference "J4") (unit 1) (value "Chassis") (footprint "Connector_Pin:Pin_D1.3mm_L11.3mm_W2.8mm_Flat")
     )
-    (path "/195f1834-ec17-48cc-80e9-521ecf0727eb"
-      (reference "J5") (unit 1) (value "+5v In Gnd") (footprint "Connector_PinHeader_2.54mm:PinHeader_1x03_P2.54mm_Vertical")
-    )
     (path "/9f18e046-a46b-4c6e-8094-d35451e925b3"
       (reference "J6") (unit 1) (value "Rx2 Tx2 Gnd") (footprint "Connector_PinHeader_2.54mm:PinHeader_1x03_P2.54mm_Vertical")
     )
+    (path "/2fa0e706-ab2e-45bb-b1b7-cdfe27c65520"
+      (reference "J?") (unit 1) (value "WAS Terminal") (footprint "TerminalBlock_TE-Connectivity:TerminalBlock_TE_282834-4_1x04_P2.54mm_Horizontal")
+    )
     (path "/c8649db0-26e8-4a89-afef-7544c6bf401e"
       (reference "R2") (unit 1) (value "1k") (footprint "Resistor_THT:R_Axial_DIN0207_L6.3mm_D2.5mm_P10.16mm_Horizontal")
@@
       (reference "R3") (unit 1) (value "1k") (footprint "Resistor_THT:R_Axial_DIN0207_L6.3mm_D2.5mm_P10.16mm_Horizontal")
     )
-    (path "/91d38898-778b-4d3c-a61c-a47d3c0c7daf"
-      (reference "R5") (unit 1) (value "1k") (footprint "Resistor_THT:R_Axial_DIN0204_L3.6mm_D1.6mm_P2.54mm_Vertical")
+    (path "/5389b411-b139-4ebf-89ee-480c9e7b113f"
+      (reference "R5") (unit 1) (value "1k") (footprint "Resistor_THT:R_Axial_DIN0207_L6.3mm_D2.5mm_P10.16mm_Horizontal")
     )
     (path "/ea61d9ea-7444-47a0-8a29-29441c5c8c96"
