File: KiCad/Steer/Steer.kicad_sch (KiCad schematic)
At the start: 41 parts, among them J2 Screw_Terminal_01x04, Q1 IRF3205, Q2 IRF3205, Q3 IRF3205, Q4 IRF3205, U1 IR2184, U2 5.0V Reg, U3 IR2184

Commit message: Steer Update
Parts:
- added C10, C9: 0.1uF, Capacitor_THT:C_Disc_D7.0mm_W2.5mm_P5.00mm, symbol Device:C_Small
- added D? (x4): 1N4007, Diode_THT:D_DO-41_SOD81_P10.16mm_Horizontal, symbol Diode:1N4007
- added J1: Switches, TerminalBlock_Phoenix:TerminalBlock_Phoenix_MKDS-1,5-4-5.08_1x04_P5.08mm_Horizontal, symbol Connector:Screw_Terminal_01x04
- added J3: Motor, TerminalBlock_Phoenix:TerminalBlock_Phoenix_MKDS-1,5-4-5.08_1x04_P5.08mm_Horizontal, symbol Connector:Screw_Terminal_01x04
- added R10, R11, R12, R13: 1k, symbol Device:R
- added U5: LTV-847, Package_DIP:DIP-16_W7.62mm, symbol Isolator:LTV-847
- U4: renamed from U?; value ACS724xLCTR-05AB -> ACS724LLCTR-10AB-T
- gave numbers to parts that had none: 10
Connections:
- net +12C: now also U4.1 (IP+), U4.2 (IP+); no longer D3.2 (A), D9.2 (A), Q1.2 (D), Q3.2 (D), U1.5 (VCC), U3.5 (VCC)
- net +5V: now also U4.8 (VCC), C10.1, R10.2, R11.2, R12.2, R13.2
- net GND: now also C10.2, C9.2, U5.11, U5.13, U5.15, U5.9
- net at C3.2, C7.2, D12.2 (A)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: now also J3.1 (Pin_1), J3.2 (Pin_2)
- net at C1.2, C2.2, D11.2 (A)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: now also J3.3 (Pin_3), J3.4 (Pin_4)
- net at U3.1 (IN): now also A1.10 (D7)
- net at U3.2 (~{SD}): now also A1.9 (D6), U1.2 (~{SD})
- net at U4.3 (IP-), U4.4 (IP-): now also D3.2 (A), D9.2 (A), Q1.2 (D), Q3.2 (D), U1.5 (VCC), U3.5 (VCC)
- net at U4.6 (FILTER): now also C9.1
- net at U4.7 (VIOUT): now also A1.19 (A0)
- net at A1.11 (D8): now also U1.1 (IN)
- net at A1.5 (D2): now also U5.10
- net at A1.6 (D3): now also U5.12
- net at A1.7 (D4): now also U5.14
- net at A1.8 (D5): now also U5.16
- new net: R13.1, U5.5
- new net: R11.1, U5.1
- new net: D?.2 (A), U5.2
- new net: R10.1, U5.7
- new net: D?.2 (A), U5.8
- new net: D?.1 (K), J1.4 (Pin_4)
- new net: D?.1 (K), J1.1 (Pin_1)
- new net: D?.1 (K), J1.2 (Pin_2)
- new net: D?.1 (K), J1.3 (Pin_3)
- new net: R12.1, U5.3
- new net: D?.2 (A), U5.4
- new net: D?.2 (A), U5.6
Other:
- title: GPS_Micro -> Steer Board
- moved on the sheet: U4

Commit message: kicad update
Parts:
- R10, R11, R12, R13: value 1k -> 180R
- gave numbers to parts that had none: 4
Changed lines of the file:
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@@
     (pin "1")
-  )
-  (symbol (lib_id "Device:R") (at 160.02 142.24 90) (unit 1)
-    (in_bom yes) (on_board yes)
-    (property "Reference" "R13" (id 0) (at 158.75 139.7 90)
-      (effects (font (size 1.27 1.27)) (justify left))
-    )
-    (property "Value" "1k" (id 1) (at 162.56 139.7 90)
-      (effects (font (size 1.27 1.27)) (justify left))
-    )
-    (property "Footprint" "" (id 2) (at 160.02 144.018 90)
-      (effects (font (size 1.27 1.27)) hide)
-    )
-    (property "Datasheet" "~" (id 3) (at 160.02 142.24 0)
-      (effects (font (size 1.27 1.27)) hide)
-    )
-    (pin "1")
-    (pin "2")
   )
   (symbol (lib_id "Device:R") (at 224.79 60.96 0) (unit 1)
@@
   (symbol (lib_id "Diode:1N4007") (at 158.75 151.13 180) (unit 1)
     (in_bom yes) (on_board yes)
-    (property "Reference" "D?" (id 0) (at 158.75 146.05 0))
+    (property "Reference" "D17" (id 0) (at 158.75 146.05 0))
     (property "Value" "1N4007" (id 1) (at 158.75 148.59 0))
     (property "Footprint" "Diode_THT:D_DO-41_SOD81_P10.16mm_Horizontal" (id 2) (at 158.75 146.685 0)
@@
     )
     (pin "1")
-  )
-  (symbol (lib_id "Device:R") (at 160.02 128.27 90) (unit 1)
-    (in_bom yes) (on_board yes)
-    (property "Reference" "R12" (id 0) (at 158.75 125.73 90)
-      (effects (font (size 1.27 1.27)) (justify left))
-    )
-    (property "Value" "1k" (id 1) (at 162.56 125.73 90)
-      (effects (font (size 1.27 1.27)) (justify left))
-    )
-    (property "Footprint" "" (id 2) (at 160.02 130.048 90)
-      (effects (font (size 1.27 1.27)) hide)
-    )
-    (property "Datasheet" "~" (id 3) (at 160.02 128.27 0)
-      (effects (font (size 1.27 1.27)) hide)
-    )
-    (pin "1")
-    (pin "2")
   )
   (symbol (lib_id "power:PWR_FLAG") (at 100.33 168.91 0) (unit 1)
@@
   (symbol (lib_id "Diode:1N4007") (at 158.75 109.22 180) (unit 1)
     (in_bom yes) (on_board yes)
-    (property "Reference" "D?" (id 0) (at 158.75 104.14 0))
+    (property "Reference" "D14" (id 0) (at 158.75 104.14 0))
     (property "Value" "1N4007" (id 1) (at 158.75 106.68 0))
     (property "Footprint" "Diode_THT:D_DO-41_SOD81_P10.16mm_Horizontal" (id 2) (at 158.75 104.775 0)
@@
       (effects (font (size 1.27 1.27)) (justify left))
     )
-    (property "Value" "1k" (id 1) (at 162.56 111.76 90)
+    (property "Value" "180R" (id 1) (at 165.1 111.76 90)
       (effects (font (size 1.27 1.27)) (justify left))
     )
@@
   (symbol (lib_id "Diode:1N4007") (at 158.75 137.16 180) (unit 1)
     (in_bom yes) (on_board yes)
-    (property "Reference" "D?" (id 0) (at 158.75 132.08 0))
+    (property "Reference" "D16" (id 0) (at 158.75 132.08 0))
     (property "Value" "1N4007" (id 1) (at 158.75 134.62 0))
     (property "Footprint" "Diode_THT:D_DO-41_SOD81_P10.16mm_Horizontal" (id 2) (at 158.75 132.715 0)
@@
   (symbol (lib_id "Diode:1N4007") (at 158.75 123.19 180) (unit 1)
     (in_bom yes) (on_board yes)
-    (property "Reference" "D?" (id 0) (at 158.75 118.11 0))
+    (property "Reference" "D15" (id 0) (at 158.75 118.11 0))
     (property "Value" "1N4007" (id 1) (at 158.75 120.65 0))
     (property "Footprint" "Diode_THT:D_DO-41_SOD81_P10.16mm_Horizontal" (id 2) (at 158.75 118.745 0)
@@
     (pin "7")
     (pin "8")
+  )
+  (symbol (lib_id "Device:R") (at 160.02 142.24 90) (unit 1)
+    (in_bom yes) (on_board yes)
+    (property "Reference" "R13" (id 0) (at 158.75 139.7 90)
+      (effects (font (size 1.27 1.27)) (justify left))
+    )
+    (property "Value" "180R" (id 1) (at 165.1 139.7 90)
+      (effects (font (size 1.27 1.27)) (justify left))
+    )
+    (property "Footprint" "" (id 2) (at 160.02 144.018 90)
+      (effects (font (size 1.27 1.27)) hide)
+    )
+    (property "Datasheet" "~" (id 3) (at 160.02 142.24 0)
+      (effects (font (size 1.27 1.27)) hide)
+    )
+    (pin "1")
+    (pin "2")
   )
   (symbol (lib_id "Isolator:LTV-847") (at 143.51 139.7 180) (unit 3)
@@
   (symbol (lib_id "power:+5V") (at 167.64 104.14 0) (unit 1)
     (in_bom yes) (on_board yes)
-    (property "Reference" "#PWR?" (id 0) (at 167.64 107.95 0)
+    (property "Reference" "#PWR05" (id 0) (at 167.64 107.95 0)
       (effects (font (size 1.27 1.27)) hide)
     )
@@
     )
     (pin "1")
+  )
+  (symbol (lib_id "Device:R") (at 160.02 128.27 90) (unit 1)
+    (in_bom yes) (on_board yes)
+    (property "Reference" "R12" (id 0) (at 158.75 125.73 90)
+      (effects (font (size 1.27 1.27)) (justify left))
+    )
+    (property "Value" "180R" (id 1) (at 165.1 125.73 90)
+      (effects (font (size 1.27 1.27)) (justify left))
+    )
+    (property "Footprint" "" (id 2) (at 160.02 130.048 90)
+      (effects (font (size 1.27 1.27)) hide)
+    )
+    (property "Datasheet" "~" (id 3) (at 160.02 128.27 0)
+      (effects (font (size 1.27 1.27)) hide)
+    )
+    (pin "1")
+    (pin "2")
   )
   (symbol (lib_id "Device:R") (at 146.05 173.99 0) (unit 1)
@@
       (effects (font (size 1.27 1.27)) (justify left))
     )
-    (property "Value" "1k" (id 1) (at 161.29 153.67 90)
+    (property "Value" "180R" (id 1) (at 163.83 153.67 90)
       (effects (font (size 1.27 1.27)) (justify left))
     )
@@
       (reference "#PWR04") (unit 1) (value "GND") (footprint "")
     )
+    (path "/babb2b10-2236-43a2-a400-1167ddd0447e"
+      (reference "#PWR05") (unit 1) (value "+5V") (footprint "")
+    )
     (path "/1e6acf8b-0742-4939-b210-97709329484b"
       (reference "#PWR06") (unit 1) (value "+12C") (footprint "")
@@
       (reference "#PWR0126") (unit 1) (value "+5V") (footprint "")
     )
-    (path "/babb2b10-2236-43a2-a400-1167ddd0447e"
-      (reference "#PWR?") (unit 1) (value "+5V") (footprint "")
-    )
     (path "/b029a6c4-c97d-4197-be8c-ac7889eee800"
       (reference "A1") (unit 1) (value "Arduino_Nano_v3.x") (footprint "Module:Arduino_Nano")
@@
       (reference "D13") (unit 1) (value "18v") (footprint "")
     )
+    (path "/50bff6d0-7c6b-4b0c-a899-d71840f71311"
+      (reference "D14") (unit 1) (value "1N4007") (footprint "Diode_THT:D_DO-41_SOD81_P10.16mm_Horizontal")
+    )
+    (path "/84c8c57a-1030-4466-abf6-d626f267e15c"
+      (reference "D15") (unit 1) (value "1N4007") (footprint "Diode_THT:D_DO-41_SOD81_P10.16mm_Horizontal")
+    )
+    (path "/7b052d84-abc1-4669-9184-92c73e851f2e"
+      (reference "D16") (unit 1) (value "1N4007") (footprint "Diode_THT:D_DO-41_SOD81_P10.16mm_Horizontal")
+    )
     (path "/284150e5-bd12-4a15-9a64-bf934cde1468"
-      (reference "D?") (unit 1) (value "1N4007") (footprint "Diode_THT:D_DO-41_SOD81_P10.16mm_Horizontal")
-    )
-    (path "/50bff6d0-7c6b-4b0c-a899-d71840f71311"
-      (reference "D?") (unit 1) (value "1N4007") (footprint "Diode_THT:D_DO-41_SOD81_P10.16mm_Horizontal")
-    )
-    (path "/7b052d84-abc1-4669-9184-92c73e851f2e"
-      (reference "D?") (unit 1) (value "1N4007") (footprint "Diode_THT:D_DO-41_SOD81_P10.16mm_Horizontal")
-    )
-    (path "/84c8c57a-1030-4466-abf6-d626f267e15c"
-      (reference "D?") (unit 1) (value "1N4007") (footprint "Diode_THT:D_DO-41_SOD81_P10.16mm_Horizontal")
+      (reference "D17") (unit 1) (value "1N4007") (footprint "Diode_THT:D_DO-41_SOD81_P10.16mm_Horizontal")
     )
     (path "/da0724b9-f9c0-47b4-af09-f03543dee5a6"
@@
       (reference "R9") (unit 1) (value "10k") (footprint "")
     )
-    (path "/e3c2d088-be20-4d25-ad4c-cde26de38a38"
-      (reference "R10") (unit 1) (value "1k") (footprint "")
+    (path "/e0f9ea92-0595-4966-a152-28b49ed50977"
+      (reference "R10") (unit 1) (value "180R") (footprint "")
     )
     (path "/5229c744-d010-44f1-bfba-3798c54b8f42"
-      (reference "R11") (unit 1) (value "1k") (footprint "")
-    )
-    (path "/488c644d-f94d-4460-a28b-8b0b8b14df2d"
-      (reference "R12") (unit 1) (value "1k") (footprint "")
-    )
-    (path "/08f5ad04-3a83-4ed0-968c-df00f6a5d225"
-      (reference "R13") (unit 1) (value "1k") (footprint "")
+      (reference "R11") (unit 1) (value "180R") (footprint "")
+    )
+    (path "/bf0b3eff-3f9d-4a99-a92a-bd40968dc993"
+      (reference "R12") (unit 1) (value "180R") (footprint "")
+    )
+    (path "/a55e089a-4c1c-4d6a-80e5-37eac5dd68ec"
+      (reference "R13") (unit 1) (value "180R") (footprint "")
     )
     (path "/d561b9e5-bac9-49c2-a7a3-3cab8d4435aa"
